File: modchip/hardware/modchip.kicad_sch (KiCad schematic)
At the start: 66 parts, among them J1 To switch T3 (I2C slave), J2 To switch T8 (GPIO46-49), J3 To switch T5 (UART0), J4 USB-C (bench use), J5 SWD, Q1 2N7002, SW1 BOOTSEL, SW2 RUN, U1 RP2354A, U2 LM66100, U3 LM66100, U4 AP2112K-3.3, U5 W25Q16JVUXIQ, U6 USBLC6-2SC6, Y1 12MHz

Commit message: modchip: route the RP2350 board and generate JLCPCB production files
Layout and routing, built by modchip/hardware/build.sh with kicad-agent-kit
(board from netlist, placement, plane fanout, Freerouting, A* finisher):

- 4 layers: F.Cu parts and signals, In1 GND, In2 +3V3, B.Cu signals; only
  the hand-soldered headers on the bottom.
- GPIOs follow the board: U1 rotated 270 puts GP11..GP0 under T3/T8 in
  header order (I2C on I2C1, GP11/GP10; T8 on GP7..GP4; UART GP0/GP1;
  reset GP27; LED GP22), so the fan-out doesn't cross.
- Hand routes laid before the router: VREG_LX and VREG_AVDD, the +3V3 trunk
  to CIN, the +1V1 DVDD pins on vias and B.Cu tracks round the exposed pad,
  the T8 fan and UART lanes, and a few boxed-in plane vias. Escape corridors
  round U1 stay clear of auto-placed parts.
- KiCad DRC: no errors, no warnings, schematic parity included.

Circuit changes on the way: no USB (SWD on J5 programs, debugs and can
power the board, the LM66100 keeping that supply out of the switch); the
RP2350A with a W25Q128JVSIQ is the default build, an RP2354A without U5/C19
the alternative; every part has an LCSC number, Basic wherever one exists,
with four in-stock Extended parts (RP2350A, LM66100, the datasheet's AOTA
inductor, the ABM8 crystal the RP2350 is tuned for); headers are not
assembled. Fixed on the way: L1's fields were passed as its DNP flag.

production/ holds the Gerber/drill zip, BOM (19 lines) and placement file
(48 parts, top side only) from the Fabrication Toolkit.

Co-Authored-By: Claude Opus 5.5 <noreply@anthropic.com>
Parts:
- removed C20, C21: 1u, Capacitor_SMD:C_0402_1005Metric, symbol Device:C
- removed J4: USB-C (bench use), Connector_USB:USB_C_Receptacle_GCT_USB4105-xx-A_16P_TopMnt_Horizontal, symbol Connector:USB_C_Receptacle_USB2.0_16P
- removed R1, R2: 5.1k, Resistor_SMD:R_0402_1005Metric, symbol Device:R
- removed R3, R4: 27, Resistor_SMD:R_0402_1005Metric, symbol Device:R
- removed R7: 1k, Resistor_SMD:R_0402_1005Metric, symbol Device:R
- removed SW1: BOOTSEL, Button_Switch_SMD:SW_Push_1P1T_NO_CK_KMR2, symbol Switch:SW_Push
- removed SW2: RUN, Button_Switch_SMD:SW_Push_1P1T_NO_CK_KMR2, symbol Switch:SW_Push
- removed U3: LM66100, Package_TO_SOT_SMD:SOT-363_SC-70-6, symbol Power_Management:LM66100DCK
- removed U4: AP2112K-3.3, Package_TO_SOT_SMD:SOT-23-5, symbol Regulator_Linear:AP2112K-3.3
- removed U6: USBLC6-2SC6, Package_TO_SOT_SMD:SOT-23-6, symbol Power_Protection:USBLC6-2SC6
- C1, C10, C11, C12, C2, C3, C4, C5, C6, C7, C8, C9: LCSC (none) -> C1525; Near (none) -> U1
- C13, C14, C15, C16: LCSC (none) -> C23733; Near (none) -> U1
- C17, C18: LCSC (none) -> C1548; Near (none) -> Y1
- C19: Fit RP2350A builds only; DNP with RP2354A -> Fitted with the RP2350A (default); leave off in an RP2354A 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; LCSC (none) -> C1525; Near (none) -> U5; now fitted
- C22: LCSC (none) -> C19702; Near (none) -> U2
- C24: LCSC (none) -> C52923; Near (none) -> U2
- D1: value green -> red; footprint LED_SMD:LED_0402_1005Metric -> LED_SMD:LED_0603_1608Metric; LCSC (none) -> C2286
- J1, J2: Note (none) -> Hand-soldered on the bottom side; not assembled (JLC: C2243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; now left out of the parts list
- J3: Note (none) -> Hand-soldered on the bottom side; not assembled (JLC: C3271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; now left out of the parts list
- J5: footprint Connector_PinHeader_1.27mm:PinHeader_1x03_P1.27mm_Vertical -> Connector_PinHeader_1.27mm:PinHeader_1x05_P1.27mm_Vertical; symbol Connector_Generic:Conn_01x03 -> Connector_Generic:Conn_01x05; Note (none) -> Debug probe: SWD, RUN, and 3.3 V for bench power (U2 blocks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; now left out of the parts list
- L1: LCSC (none) -> C42411119; MPN (none) -> Abracon AOTA-B201610S3R3-101-T, the datasheet's choice (che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; now fitted
- Q1: LCSC (none) -> C8545
- R10, R11, R12, R13, R14, R15, R16, R17, R18, R19: LCSC (none) -> C25076
- R20, R21: LCSC (none) -> C25900; Near (none) -> J1
- R22, R23: LCSC (none) -> C25741; Near (none) -> U1
- R24: LCSC (none) -> C25741; Near (none) -> Q1
- R25: LCSC (none) -> C11702; Near (none) -> Q1
- R5: LCSC (none) -> C25105
- R6: LCSC (none) -> C11702; Near (none) -> Y1
- R8: LCSC (none) -> C25744; Near (none) -> J5
- R9: LCSC (none) -> C25104; Near (none) -> D1
- TP1: now left out of the parts list
- U1: value RP2354A -> RP2350A; footprint Package_DFN_QFN:QFN-60-1EP_7x7mm_P0.4mm_EP3.4x3.4mm -> Package_DFN_QFN:QFN-60-1EP_7x7mm_P0.4mm_EP3.4x3.4mm_ThermalVias; symbol MCU_RaspberryPi:RP2354A -> MCU_RaspberryPi:RP2350A; LCSC (none) -> C42411118; Variant (none) -> RP2354A (2 MiB in package): same footprint and pinout; then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
- U2: LCSC (none) -> C2869734
- U5: value W25Q16JVUXIQ -> W25Q128JVSIQ; footprint Package_SON:Winbond_USON-8-1EP_3x2mm_P0.5mm_EP0.2x1.6mm -> Package_SO:SOIC-8_5.3x5.3mm_P1.27mm; symbol Memory_Flash:W25Q16JVSS -> Memory_Flash:W25Q128JVS; Fit RP2350A builds only; DNP with RP2354A -> Fitted with the RP2350A (default); leave off in an RP2354A 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; LCSC (none) -> C97521; Note (none) -> W25Q128JVSIQ, 16 MiB, JLCPCB Basic; any 208-mil SOIC-8 QSPI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; now fitted
- Y1: LCSC (none) -> C20625731; MPN Abracon ABM8-272-T3 -> Abracon ABM8-272-T3: the RP2350 is tuned for it (10 pF load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
Connections:
- net +3V3: now also J5.1 (Pin_1)
- net GND: now also J5.3 (Pin_3); no longer J5.2 (Pin_2)
- net I2C_SCL: now also U1.15 (GPIO11); no longer U1.8 (GPIO5)
- net I2C_SDA: now also U1.14 (GPIO10); no longer U1.7 (GPIO4)
- net RESET_DRV: now also U1.41 (GPIO27/ADC1); no longer U1.16 (GPIO12)
- net RUN: now also J5.5 (Pin_5)
- net SWCLK: now also J5.2 (Pin_2); no longer J5.1 (Pin_1)
- net SWDIO: now also J5.4 (Pin_4); no longer J5.3 (Pin_3)
- net T3_SPI_CS: now also U1.12 (GPIO8); no longer U1.10 (GPIO7)
- net T3_SPI_DO: now also U1.13 (GPIO9); no longer U1.9 (GPIO6)
- net T8_GPIO46: now also U1.10 (GPIO7); no longer U1.12 (GPIO8)
- net T8_GPIO47: now also U1.8 (GPIO5); no longer U1.13 (GPIO9)
- net T8_GPIO48: now also U1.9 (GPIO6); no longer U1.14 (GPIO10)
- net T8_GPIO49: now also U1.7 (GPIO4); no longer U1.15 (GPIO11)
- net LED: now reaches U1.34 (GPIO22)
- net LED: now also R9.1
- net LED_GP25: no longer names the net of U1.37 (GPIO25)
- net LED_GP25: no longer R9.1
- net USB_DM: no longer names the net of U1.51 (USB_DM)
- net USB_DP: no longer names the net of U1.52 (USB_DP)
- no-connect marks 25 -> 22
Other:
- note added: "FLASH, CLOCK, DEBUG U5/C19: fitted with the RP2350A, left off with an RP2354A. Programming and debug are over SWD (J5); there is no USB."
- note added: "MCU Default build: RP2350A with U5, a W25Q128JVSIQ (16 MiB). Alternative: RP2354A (2 MiB in the package, same pinout) with U5 and C19 left off. Never fit U5 with an RP2354A: both flash chips would answer on QSPI_SS."
- note added: "POWER The board runs from the switch's 3.3 V (T3/T8 pin 4) through the ideal diode U2. On the bench a debug probe can supply 3.3 V on J5 pin 1 instead; U2 keeps it out of the switch. SW_SENSE tells the firmware whether the switch is on: until it is, keep every switch-facing pin high-impedance with its input buffer off."
- note removed: "FLASH, CLOCK, BOOT, DEBUG U5/C19: DNP with the RP2354A. Keep the QSPI stubs to U5 short."
- note removed: "MCU RP2354A: RP2350A with 2 MiB of flash in the package (same pinout). With an RP2350A, fit U5 and C19. Never fit U5 with an RP2354A: both would answer on QSPI_SS."
- note removed: "POWER The switch's 3.3 V (T3/T8 pin 4) and USB's 3.3 V are ORed by two ideal diodes, so neither back-feeds the other. SW_SENSE tells the firmware whether the switch is on: until it is, keep every switch-facing pin high-impedance with its input buffer off."
